File: PCB_Shield/Arduino_Uno.kicad_sch (KiCad schematic)
At the start: 4 parts, among them J1 Power, J2 Digital/PWM, J3 Analog, J4 Digital/PWM

Commit message: holes insted of pads for soldering
Connections:
- net SCL/A5 renamed A5
- net A5: no longer J2.1 (Pin_1)
- net SDA/A4 renamed A4
- net A4: no longer J2.2 (Pin_2)
- new net SCL: J2.1 (Pin_1)
- new net SDA: J2.2 (Pin_2)
Changed lines of the file:
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@@
 		)
 	)
-	(label "SDA{slash}A4"
+	(label "SDA"
 		(at 74.93 29.21 180)
 		(fields_autoplaced yes)
@@
 		)
 	)
-	(label "SCL{slash}A5"
+	(label "SCL"
 		(at 74.93 26.67 180)
 		(fields_autoplaced yes)
@@
 		)
 	)
-	(label "SDA{slash}A4"
+	(label "A4"
 		(at 21.59 69.85 0)
 		(fields_autoplaced yes)
@@
 		)
 	)
-	(label "SCL{slash}A5"
+	(label "A5"
 		(at 21.59 72.39 0)
 		(fields_autoplaced yes)
